Commit message: add kinect plugin in urdf and python interface

File: my_arm/urdf/my_arm_backup.urdf (robot description, URDF)
Before this commit: robot my_arm, 9 links, 8 joints
Links:
- removed link camera_link
- removed link finger_link1
- removed link finger_link2
- link base: mass 0.001 -> 1
- link elbow_link: mass 0.001 -> 1
- link gripper_link: mass 0.0005 -> 1
- link hand_link: mass 0.001 -> 1
- link wrist_link: mass 0.001 -> 1
Joints:
- removed joint camera_joint
- removed joint finger_joint1
- removed joint finger_joint2
