Commit message: new urdf

File: my_arm/urdf/my_arm.urdf (robot description, URDF)
Before this commit: robot my_arm, 3 links, 2 joints
Links:
- removed link Link1
- removed link Link2
- added link base; visual mesh filename=package://my_arm/meshes/platform.stl scale=0.001 0.001 0.001
- added link elbow_link; visual mesh filename=package://my_arm/meshes/arm_1.stl scale=0.001 0.001 0.001
- added link finger_link1; visual mesh filename=package://my_arm/meshes/finger_1.stl scale=0.001 0.001 0.001
- added link finger_link2; visual mesh filename=package://my_arm/meshes/finger_2.stl scale=0.001 0.001 0.001
- added link gripper_link; visual mesh filename=package://my_arm/meshes/hand.stl scale=0.001 0.001 0.001
- added link hand_link; visual mesh filename=package://my_arm/meshes/carpus.stl scale=0.001 0.001 0.001
- added link wrist_link; visual mesh filename=package://my_arm/meshes/arm_2.stl scale=0.001 0.001 0.001
- link base_link: mass 0.579526073390066 -> None; geometry 
Joints:
- removed joint Join1
- removed joint Joint2
- added joint base2base_joint: type revolute, parent base_link, child base, origin xyz=0 0 0 rpy=0 0 0, axis 0 0 1, limit lower=-1.570795 upper=1.570795 effort=30 velocity=1.0
- added joint base_joint: type revolute, parent base, child elbow_link, origin xyz=0.190 0.198 0.243 rpy=0 0 0, axis 1 0 0, limit lower=-1.570795 upper=1.570795 effort=30 velocity=1.0
- added joint elbow_joint: type revolute, parent elbow_link, child wrist_link, origin xyz=0.371 0.104 0.520 rpy=0 0 0, axis 1 0 0, limit lower=-1.570795 upper=1.570795 effort=30 velocity=1.0
- added joint finger_joint1: type revolute, parent gripper_link, child finger_link1, origin xyz=1.116 0.125 0.526 rpy=0 0 0, axis 1 0 0, limit lower=-1.570795 upper=1.570795 effort=30 velocity=1.0
- added joint finger_joint2: type revolute, parent gripper_link, child finger_link2, origin xyz=1.116 0.184 0.526 rpy=0 0 0, axis 1 0 0, limit lower=-1.570795 upper=1.570795 effort=30 velocity=1.0
- added joint hand_joint: type revolute, parent hand_link, child gripper_link, origin xyz=0.861 0.118 0.454 rpy=0 0 0, axis 1 0 0, limit lower=-1.570795 upper=1.570795 effort=30 velocity=1.0
- added joint wrist_joint: type revolute, parent wrist_link, child hand_link, origin xyz=0.842 0.099 0.441 rpy=0 0 0, axis 1 0 0, limit lower=-1.570795 upper=1.570795 effort=30 velocity=1.0

Commit message: model2.0

File: my_arm/urdf/my_arm.urdf (robot description, URDF)
Before this commit: robot my_arm, 8 links, 7 joints
Joints:
- joint base2base_joint: limit lower=-1.570795 upper=1.570795 effort=30 velocity=1.0 -> (none); origin xyz=0 0 0 rpy=0 0 0 -> xyz=0.137 0.134 0 rpy=0 0 0; type revolute -> continuous
- joint base_joint: axis 1 0 0 -> 0 1 0; origin xyz=0.190 0.198 0.243 rpy=0 0 0 -> xyz=0.053 0.064 0.243 rpy=0 0 0
- joint elbow_joint: axis 1 0 0 -> 0 1 0; origin xyz=0.371 0.104 0.520 rpy=0 0 0 -> xyz=0.181 -0.094 0.277 rpy=0 0 0
- joint finger_joint1: axis 1 0 0 -> 0 0 1; origin xyz=1.116 0.125 0.526 rpy=0 0 0 -> xyz=0.155 0.007 0.052 rpy=0 0 0
- joint finger_joint2: axis 1 0 0 -> 0 0 1; origin xyz=1.116 0.184 0.526 rpy=0 0 0 -> xyz=0.155 0.059 0.052 rpy=0 0 0
- joint hand_joint: origin xyz=0.861 0.118 0.454 rpy=0 0 0 -> xyz=0.019 0.019 0.013 rpy=0 0 0; type revolute -> continuous
- joint wrist_joint: axis 1 0 0 -> 0 1 0; origin xyz=0.842 0.099 0.441 rpy=0 0 0 -> xyz=0.471 -0.005 -0.079 rpy=0 0 0

Commit message: arm can attach object now

File: my_arm/urdf/my_arm.urdf (robot description, URDF)
Before this commit: robot my_arm, 9 links, 8 joints
Links:
- added link end, mass 0.001
- added link support, mass 0.001; collision box size=0.1 0.1 1.5; visual box size=0.1 0.1 1.5
Joints:
- added joint end_joint: type revolute, parent gripper_link, child end, origin xyz=0 0 0.184 rpy=0 0 0, axis 0 1 0, limit lower=-1.570795 upper=1.570795 effort=30 velocity=1.0
- added joint support_joint: type fixed, parent world, child support, origin xyz=0 0 0 rpy=0 0 0, axis 0 0 1
- joint base2base_joint: origin xyz=0.137 0.137 0 rpy=0 0 0 -> xyz=0 -0.05 1.3 rpy=1.5707963 0 0; parent world -> support
- joint camera_joint: origin xyz=0.35 0.137 0.1 rpy=0 0 0 -> xyz=0 0 1.55 rpy=0 0 0
- joint elbow_joint: limit lower=-1.570795 upper=1.570795 effort=30 velocity=1.0 -> lower=-3.1415926 upper=3.1415926 effort=30 velocity=1.0
- joint wrist_joint: limit lower=-1.570795 upper=1.570795 effort=30 velocity=1.0 -> lower=-3.1415926 upper=3.1415926 effort=30 velocity=1.0
